File: board/TOFE-AXIOM-adapter.sch (KiCad schematic (older format))
At the start: 2 parts, among them U1 TOFE-8X, U2 TOFE-8X

Commit message: Slowly working on the adapter.
Parts:
- removed U2: TOFE-8X, ~, symbol TOFE-8X
- added NORTH1, SOUTH1: AXIOM-PCIE, symbol AXIOM-PCIE
Connections:
- net labels added: +5V, N_IO0, N_IO1, N_IO2, N_IO3, N_IO4, N_IO5, N_IO6, N_IO7, N_LVDS_A0, N_LVDS_A1, N_LVDS_A2, N_LVDS_A3, N_LVDS_A4, N_LVDS_A5, N_LVDS_B0, N_LVDS_B1, N_LVDS_B2, N_LVDS_B3, N_LVDS_B4, N_LVDS_B5, N_SCL, N_SDA, SMCLK, SMDAT, S_IO0, S_IO1, S_IO2, S_IO3, S_IO4, S_IO5, S_IO6, S_IO7, S_LVDS_A0, S_LVDS_A1, S_LVDS_A2, S_LVDS_A3, S_LVDS_A4, S_LVDS_A5, S_LVDS_B0, S_LVDS_B1, S_LVDS_B2, S_LVDS_B3, S_LVDS_B4, S_LVDS_B5, S_SCL, S_SDA
- net labels removed: A13, A14, A16, A17, A19, A21, A22, A25, A26, A29, A30, A32, A33, A35, A36, A39, A40, A43, A44, A47, A48, A5, A6, A7, A8, B11, B12, B14, B15, B19, B20, B23, B24, B27, B28, B30, B33, B34, B37, B38, B41, B42, B45, B46, B5, B6, B9
- wire segments 312 -> 151
- no-connect marks 0 -> 1
Other:
- note added: "apertus AXIOM Connector"
- note removed: "TOFE 8x Connector"

Commit message: More work.
Parts:
- removed SOUTH1: AXIOM-PCIE, symbol AXIOM-PCIE
- added C1: C, symbol C
- added R1: R, symbol R
Connections:
- net labels added: VCC_3V3, VCC_5V0
- net labels removed: +5V
- wire segments 151 -> 207
Changed lines of the file:
@@
 Comment4 ""
 $EndDescr
-Text Label 4950 8450 2    60   ~ 12
-GND
 Text Label 6210 2950 2    60   ~ 12
 S_IO7
@@
 	1    0    0    -1
 $EndComp
-$Comp
-L AXIOM-PCIE SOUTH1
-U 1 1 56EB9DF7
-P 10340 8060
-F 0 "SOUTH1" H 10240 8510 60  0000 C CNN
-F 1 "AXIOM-PCIE" H 9490 8510 60  0000 C CNN
-F 2 "" H 8240 8160 60  0000 C CNN
-F 3 "" H 8240 8160 60  0000 C CNN
-	1    10340 8060
-	1    0    0    -1
-$EndComp
 NoConn ~ 5600 6150
 Wire Wire Line
 	3900 2850 3800 2850
 Wire Wire Line
-	3800 2850 3800 8300
+	3800 2850 3800 3150
+Wire Wire Line
+	3800 3150 3800 3950
+Wire Wire Line
+	3800 3950 3800 4250
+Wire Wire Line
+	3800 4250 3800 4450
+Wire Wire Line
+	3800 4450 3800 4850
+Wire Wire Line
+	3800 4850 3800 4950
+Wire Wire Line
+	3800 4950 3800 5250
+Wire Wire Line
+	3800 5250 3800 5350
+Wire Wire Line
+	3800 5350 3800 5650
+Wire Wire Line
+	3800 5650 3800 5950
+Wire Wire Line
+	3800 5950 3800 6350
+Wire Wire Line
+	3800 6350 3800 6450
+Wire Wire Line
+	3800 6450 3800 6750
+Wire Wire Line
+	3800 6750 3800 6850
+Wire Wire Line
+	3800 6850 3800 7150
+Wire Wire Line
+	3800 7150 3800 7250
+Wire Wire Line
+	3800 7250 3800 7550
+Wire Wire Line
+	3800 7550 3800 7750
+Wire Wire Line
+	3800 7750 3800 8300
 Wire Wire Line
 	3800 3150 3900 3150
@@
 	5600 2850 5700 2850
 Wire Wire Line
-	5700 2850 5700 8300
+	5700 2850 5700 3850
+Wire Wire Line
+	5700 3850 5700 4150
+Wire Wire Line
+	5700 4150 5700 4450
+Wire Wire Line
+	5700 4450 5700 4750
+Wire Wire Line
+	5700 4750 5700 5050
+Wire Wire Line
+	5700 5050 5700 5150
+Wire Wire Line
+	5700 5150 5700 5450
+Wire Wire Line
+	5700 5450 5700 5550
+Wire Wire Line
+	5700 5550 5700 5850
+Wire Wire Line
+	5700 5850 5700 6250
+Wire Wire Line
+	5700 6250 5700 6550
+Wire Wire Line
+	5700 6550 5700 6650
+Wire Wire Line
+	5700 6650 5700 6950
+Wire Wire Line
+	5700 6950 5700 7050
+Wire Wire Line
+	5700 7050 5700 7350
+Wire Wire Line
+	5700 7350 5700 7450
+Wire Wire Line
+	5700 7450 5700 7750
+Wire Wire Line
+	5700 7750 5700 8300
 Wire Wire Line
 	5700 4150 5600 4150
@@
 Connection ~ 5700 7450
 Wire Wire Line
-	5700 8300 3800 8300
+	5700 8300 4700 8300
+Wire Wire Line
+	4700 8300 3800 8300
 Connection ~ 3800 7750
 Connection ~ 5700 7750
 Wire Wire Line
-	4700 8300 4700 8450
+	4700 8300 4700 8350
 Connection ~ 4700 8300
 Wire Wire Line
@@
 	3700 3450 3900 3450
 Wire Wire Line
-	3700 2300 3700 3450
+	3700 2300 3700 3250
+Wire Wire Line
+	3700 3250 3700 3450
 Wire Wire Line
 	3700 3250 3900 3250
@@
 	5600 3350 5800 3350
 Wire Wire Line
-	5800 2300 5800 3450
+	5800 2300 5800 3350
+Wire Wire Line
+	5800 3350 5800 3450
 Wire Wire Line
 	5800 3450 5600 3450
 Wire Wire Line
-	3700 2300 5800 2300
+	3700 2300 4850 2300
+Wire Wire Line
+	4850 2300 5800 2300
 Connection ~ 5800 3350
 Connection ~ 3700 3250
@@
 	3850 2750 3900 2750
 Wire Wire Line
-	3850 2400 3850 2750
+	3850 2400 3850 2550
+Wire Wire Line
+	3850 2550 3850 2650
+Wire Wire Line
+	3850 2650 3850 2750
 Wire Wire Line
 	3850 2650 3900 2650
@@
 	5650 2750 5600 2750
 Wire Wire Line
-	5650 2400 5650 2750
+	5650 2400 5650 2650
+Wire Wire Line
+	5650 2650 5650 2750
 Wire Wire Line
 	5650 2650 5600 2650
 Wire Wire Line
-	3850 2400 5650 2400
+	3850 2400 5150 2400
+Wire Wire Line
+	5150 2400 5650 2400
 Connection ~ 5650 2650
 Connection ~ 3850 2550
@@
 	5150 2200 5450 2200
 Connection ~ 5150 2400
-Wire Wire Line
-	4700 8450 4950 8450
 Wire Wire Line
 	5600 3550 6210 3550
@@
 	10740 2390 10780 2390
 Wire Wire Line
-	10780 2390 10780 4720
+	10780 2390 10780 2690
+Wire Wire Line
+	10780 2690 10780 2990
+Wire Wire Line
+	10780 2990 10780 3290
+Wire Wire Line
+	10780 3290 10780 3690
+Wire Wire Line
+	10780 3690 10780 3990
+Wire Wire Line
+	10780 3990 10780 4290
+Wire Wire Line
+	10780 4290 10780 4720
 Wire Wire Line
 	10740 2690 10780 2690
@@
 Connection ~ 10780 3690
 Wire Wire Line
-	10780 4720 9010 4720
+	10780 4720 9940 4720
+Wire Wire Line
+	9940 4720 9010 4720
 Connection ~ 10780 4290
 Wire Wire Line
 	9040 4290 9010 4290
 Wire Wire Line
-	9010 4720 9010 3990
+	9010 4720 9010 4290
+Wire Wire Line
+	9010 4290 9010 3990
 Wire Wire Line
 	9010 3990 9040 3990
 Connection ~ 9010 4290
 $Comp
-L GND #PWR?
+L GND #PWR1
 U 1 1 56EBC288
 P 9940 4780
-F 0 "#PWR?" H 9940 4530 50  0001 C CNN
+F 0 "#PWR1" H 9940 4530 50  0001 C CNN
 F 1 "GND" H 9940 4630 50  0000 C CNN
 F 2 "" H 9940 4780 50  0000 C CNN
@@
 	9940 4780 9940 4720
 Connection ~ 9940 4720
+Wire Wire Line
+	8490 3690 9040 3690
+Text Label 8490 3690 0    60   ~ 0
+VCC_5V0
+Text Label 8490 2590 0    60   ~ 0
+VCC_3V3
+Wire Wire Line
+	10740 3390 10980 3390
 $Comp
-L +5V #PWR?
-U 1 1 56EBC38D
-P 8980 3690
-F 0 "#PWR?" H 8980 3540 50  0001 C CNN
-F 1 "+5V" H 8980 3830 50  0000 C CNN
-F 2 "" H 8980 3690 50  0000 C CNN
-F 3 "" H 8980 3690 50  0000 C CNN
-	1    8980 3690
+L R R1
+U 1 1 56EBC757
+P 11180 3280
+F 0 "R1" V 11260 3280 50  0000 C CNN
+F 1 "R" V 11180 3280 50  0000 C CNN
+F 2 "" V 11110 3280 50  0000 C CNN
+F 3 "" H 11180 3280 50  0000 C CNN
+	1    11180 3280
+	0    1    1    0
+$EndComp
+$Comp
+L C C1
+U 1 1 56EBC822
+P 11190 3500
+F 0 "C1" H 11215 3600 50  0000 L CNN
+F 1 "C" H 11215 3400 50  0000 L CNN
+F 2 "" H 11228 3350 50  0000 C CNN
+F 3 "" H 11190 3500 50  0000 C CNN
+	1    11190 3500
+	0    1    1    0
+$EndComp
+Wire Wire Line
+	10980 3500 11040 3500
+Wire Wire Line
+	10980 3280 10980 3390
+Wire Wire Line
+	10980 3390 10980 3500
+Wire Wire Line
+	10980 3280 11030 3280
+Connection ~ 10980 3390
+$Comp
+L GND #PWR2
+U 1 1 56EBCC2F
+P 11440 3500
+F 0 "#PWR2" H 11440 3250 50  0001 C CNN
+F 1 "GND" H 11440 3350 50  0000 C CNN
+F 2 "" H 11440 3500 50  0000 C CNN
+F 3 "" H 11440 3500 50  0000 C CNN
+	1    11440 3500
 	1    0    0    -1
 $EndComp
 Wire Wire Line
-	8980 3690 9040 3690
+	11440 3500 11340 3500
+$Comp
+L GND #PWR?
+U 1 1 56EBCF33
+P 4700 8350
+F 0 "#PWR?" H 4700 8100 50  0001 C CNN
+F 1 "GND" H 4700 8200 50  0000 C CNN
+F 2 "" H 4700 8350 50  0000 C CNN
+F 3 "" H 4700 8350 50  0000 C CNN
+	1    4700 8350
+	1    0    0    -1
+$EndComp
 $EndSCHEMATC

Commit message: Import PCI-Express connectors.
Connections:
- wire segments 207 -> 155
Changed lines of the file:
@@
 	3900 2850 3800 2850
 Wire Wire Line
-	3800 2850 3800 3150
-Wire Wire Line
-	3800 3150 3800 3950
-Wire Wire Line
-	3800 3950 3800 4250
-Wire Wire Line
-	3800 4250 3800 4450
-Wire Wire Line
-	3800 4450 3800 4850
-Wire Wire Line
-	3800 4850 3800 4950
-Wire Wire Line
-	3800 4950 3800 5250
-Wire Wire Line
-	3800 5250 3800 5350
-Wire Wire Line
-	3800 5350 3800 5650
-Wire Wire Line
-	3800 5650 3800 5950
-Wire Wire Line
-	3800 5950 3800 6350
-Wire Wire Line
-	3800 6350 3800 6450
-Wire Wire Line
-	3800 6450 3800 6750
-Wire Wire Line
-	3800 6750 3800 6850
-Wire Wire Line
-	3800 6850 3800 7150
-Wire Wire Line
-	3800 7150 3800 7250
-Wire Wire Line
-	3800 7250 3800 7550
-Wire Wire Line
-	3800 7550 3800 7750
-Wire Wire Line
-	3800 7750 3800 8300
+	3800 2850 3800 8300
 Wire Wire Line
 	3800 3150 3900 3150
@@
 	5600 2850 5700 2850
 Wire Wire Line
-	5700 2850 5700 3850
-Wire Wire Line
-	5700 3850 5700 4150
-Wire Wire Line
-	5700 4150 5700 4450
-Wire Wire Line
-	5700 4450 5700 4750
-Wire Wire Line
-	5700 4750 5700 5050
-Wire Wire Line
-	5700 5050 5700 5150
-Wire Wire Line
-	5700 5150 5700 5450
-Wire Wire Line
-	5700 5450 5700 5550
-Wire Wire Line
-	5700 5550 5700 5850
-Wire Wire Line
-	5700 5850 5700 6250
-Wire Wire Line
-	5700 6250 5700 6550
-Wire Wire Line
-	5700 6550 5700 6650
-Wire Wire Line
-	5700 6650 5700 6950
-Wire Wire Line
-	5700 6950 5700 7050
-Wire Wire Line
-	5700 7050 5700 7350
-Wire Wire Line
-	5700 7350 5700 7450
-Wire Wire Line
-	5700 7450 5700 7750
-Wire Wire Line
-	5700 7750 5700 8300
+	5700 2850 5700 8300
 Wire Wire Line
 	5700 4150 5600 4150
@@
 Connection ~ 5700 7450
 Wire Wire Line
-	5700 8300 4700 8300
-Wire Wire Line
-	4700 8300 3800 8300
+	5700 8300 3800 8300
 Connection ~ 3800 7750
 Connection ~ 5700 7750
@@
 	3700 3450 3900 3450
 Wire Wire Line
-	3700 2300 3700 3250
-Wire Wire Line
-	3700 3250 3700 3450
+	3700 2300 3700 3450
 Wire Wire Line
 	3700 3250 3900 3250
@@
 	5600 3350 5800 3350
 Wire Wire Line
-	5800 2300 5800 3350
-Wire Wire Line
-	5800 3350 5800 3450
+	5800 2300 5800 3450
 Wire Wire Line
 	5800 3450 5600 3450
 Wire Wire Line
-	3700 2300 4850 2300
-Wire Wire Line
-	4850 2300 5800 2300
+	3700 2300 5800 2300
 Connection ~ 5800 3350
 Connection ~ 3700 3250
@@
 	3850 2750 3900 2750
 Wire Wire Line
-	3850 2400 3850 2550
-Wire Wire Line
-	3850 2550 3850 2650
-Wire Wire Line
-	3850 2650 3850 2750
+	3850 2400 3850 2750
 Wire Wire Line
 	3850 2650 3900 2650
@@
 	5650 2750 5600 2750
 Wire Wire Line
-	5650 2400 5650 2650
-Wire Wire Line
-	5650 2650 5650 2750
+	5650 2400 5650 2750
 Wire Wire Line
 	5650 2650 5600 2650
 Wire Wire Line
-	3850 2400 5150 2400
-Wire Wire Line
-	5150 2400 5650 2400
+	3850 2400 5650 2400
 Connection ~ 5650 2650
 Connection ~ 3850 2550
@@
 	10740 2390 10780 2390
 Wire Wire Line
-	10780 2390 10780 2690
-Wire Wire Line
-	10780 2690 10780 2990
-Wire Wire Line
-	10780 2990 10780 3290
-Wire Wire Line
-	10780 3290 10780 3690
-Wire Wire Line
-	10780 3690 10780 3990
-Wire Wire Line
-	10780 3990 10780 4290
-Wire Wire Line
-	10780 4290 10780 4720
+	10780 2390 10780 4720
 Wire Wire Line
 	10740 2690 10780 2690
@@
 Connection ~ 10780 3690
 Wire Wire Line
-	10780 4720 9940 4720
-Wire Wire Line
-	9940 4720 9010 4720
+	10780 4720 9010 4720
 Connection ~ 10780 4290
 Wire Wire Line
 	9040 4290 9010 4290
 Wire Wire Line
-	9010 4720 9010 4290
-Wire Wire Line
-	9010 4290 9010 3990
+	9010 4720 9010 3990
 Wire Wire Line
 	9010 3990 9040 3990
 Connection ~ 9010 4290
 $Comp
-L GND #PWR1
+L GND #PWR01
 U 1 1 56EBC288
 P 9940 4780
-F 0 "#PWR1" H 9940 4530 50  0001 C CNN
+F 0 "#PWR01" H 9940 4530 50  0001 C CNN
 F 1 "GND" H 9940 4630 50  0000 C CNN
 F 2 "" H 9940 4780 50  0000 C CNN
@@
 	10980 3500 11040 3500
 Wire Wire Line
-	10980 3280 10980 3390
-Wire Wire Line
-	10980 3390 10980 3500
+	10980 3280 10980 3500
 Wire Wire Line
 	10980 3280 11030 3280
 Connection ~ 10980 3390
 $Comp
-L GND #PWR2
+L GND #PWR02
 U 1 1 56EBCC2F
 P 11440 3500
-F 0 "#PWR2" H 11440 3250 50  0001 C CNN
+F 0 "#PWR02" H 11440 3250 50  0001 C CNN
 F 1 "GND" H 11440 3350 50  0000 C CNN
 F 2 "" H 11440 3500 50  0000 C CNN
@@
 	11440 3500 11340 3500
 $Comp
-L GND #PWR?
+L GND #PWR03
 U 1 1 56EBCF33
 P 4700 8350
-F 0 "#PWR?" H 4700 8100 50  0001 C CNN
+F 0 "#PWR03" H 4700 8100 50  0001 C CNN
 F 1 "GND" H 4700 8200 50  0000 C CNN
 F 2 "" H 4700 8350 50  0000 C CNN

Commit message: Slowly getting there.
Parts:
- C1: footprint (none) -> Capacitors_SMD:C_1206_HandSoldering
- NORTH1: footprint (none) -> w_conn_pc:pci-x_conn-x1
- R1: footprint (none) -> Resistors_SMD:R_0603_HandSoldering
- U1: footprint ~ -> TOFE_8X_HalfHeight:TOFE_8X_HalfHeight
Changed lines of the file:
@@
 F 0 "U1" H 5200 2400 60  0000 C CNN
 F 1 "TOFE-8X" H 4550 2400 60  0000 C CNN
-F 2 "~" H 3900 4950 60  0000 C CNN
+F 2 "TOFE_8X_HalfHeight:TOFE_8X_HalfHeight" H 3900 4950 60  0001 C CNN
 F 3 "~" H 3900 4950 60  0000 C CNN
 	1    5200 5250
@@
 F 0 "NORTH1" H 10240 5540 60  0000 C CNN
 F 1 "AXIOM-PCIE" H 9490 5540 60  0000 C CNN
-F 2 "" H 8240 5190 60  0000 C CNN
+F 2 "w_conn_pc:pci-x_conn-x1" H 8240 5190 60  0001 C CNN
 F 3 "" H 8240 5190 60  0000 C CNN
 	1    10340 5090
@@
 F 0 "R1" V 11260 3280 50  0000 C CNN
 F 1 "R" V 11180 3280 50  0000 C CNN
-F 2 "" V 11110 3280 50  0000 C CNN
+F 2 "Resistors_SMD:R_0603_HandSoldering" V 11110 3280 50  0001 C CNN
 F 3 "" H 11180 3280 50  0000 C CNN
 	1    11180 3280
@@
 F 0 "C1" H 11215 3600 50  0000 L CNN
 F 1 "C" H 11215 3400 50  0000 L CNN
-F 2 "" H 11228 3350 50  0000 C CNN
+F 2 "Capacitors_SMD:C_1206_HandSoldering" H 11228 3350 50  0001 C CNN
 F 3 "" H 11190 3500 50  0000 C CNN
 	1    11190 3500
