File: board/TOFE-AXIOM-adapter.kicad_pcb (KiCad board)
At the start: 4 copper layers, 68.9 x 31.9 mm, 21 parts, among them CN1 C, U1 24AA01/24LC01B, U2 LM317T, U3 LM7805CT

Commit message: More DRC fixing.
Routing:
- net /VCC3V3: track 95.1 -> 100.0 mm
- net /PRSTN: track 71.5 -> 71.0 mm
Changed lines of the file:
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@@
   (general
     (links 250)
-    (no_connects 5)
+    (no_connects 0)
     (area 162.059499 156.057599 231.355901 188.340501)
     (thickness 1.6)
     (drawings 25)
-    (tracks 5735)
+    (tracks 5745)
     (zones 0)
     (modules 21)
@@
   )
   (layers
-    (0 F.Cu signal hide)
+    (0 F.Cu signal)
     (1 In1.Cu signal hide)
-    (2 In2.Cu signal)
-    (31 B.Cu signal hide)
+    (2 In2.Cu signal hide)
+    (31 B.Cu signal)
     (32 B.Adhes user)
     (33 F.Adhes user)
@@
   (segment (start 225.306682 177.2) (end 231.15 177.2) (width 0.1524) (layer B.Cu) (net 0))
   (segment (start 231.15 177.2) (end 231.15 177.3) (width 0.1524) (layer B.Cu) (net 0))
-  (segment (start 175.126069 179.04) (end 174.80278 179.04) (width 0.1524) (layer F.Cu) (net 1))
-  (segment (start 180.34 178.7398) (end 180.0398 179.04) (width 0.1524) (layer F.Cu) (net 1))
-  (segment (start 174.69922 184.44874) (end 174.69922 179.14356) (width 0.1524) (layer B.Cu) (net 1))
-  (via (at 174.80278 179.04) (size 0.4572) (drill 0.254) (layers F.Cu B.Cu) (net 1))
-  (segment (start 174.69922 179.14356) (end 174.80278 179.04) (width 0.1524) (layer B.Cu) (net 1))
-  (segment (start 180.0398 179.04) (end 175.126069 179.04) (width 0.1524) (layer F.Cu) (net 1))
+  (segment (start 175.031401 179.679613) (end 175.26 179.451014) (width 0.1524) (layer B.Cu) (net 1))
+  (segment (start 175.971214 178.7398) (end 175.488599 179.222415) (width 0.1524) (layer F.Cu) (net 1))
+  (segment (start 180.34 178.7398) (end 175.971214 178.7398) (width 0.1524) (layer F.Cu) (net 1))
+  (segment (start 174.69922 180.011794) (end 175.031401 179.679613) (width 0.1524) (layer B.Cu) (net 1))
+  (segment (start 174.69922 184.44874) (end 174.69922 180.011794) (width 0.1524) (layer B.Cu) (net 1))
+  (segment (start 175.488599 179.222415) (end 175.26 179.451014) (width 0.1524) (layer F.Cu) (net 1))
+  (via (at 175.26 179.451014) (size 0.4572) (drill 0.254) (layers F.Cu B.Cu) (net 1))
   (segment (start 216.53 181.39) (end 219.906711 181.39) (width 0.1524) (layer F.Cu) (net 1))
   (segment (start 220.2386 181.3814) (end 220.23 181.39) (width 0.1524) (layer B.Cu) (net 1))
@@
   (segment (start 223.69882 182.49713) (end 222.58309 181.3814) (width 0.1524) (layer F.Cu) (net 1))
   (segment (start 184.6992 187.25036) (end 184.6992 184.94912) (width 0.1524) (layer B.Cu) (net 2))
-  (segment (start 175.26 172.72) (end 175.26 180.34) (width 0.1524) (layer In2.Cu) (net 3))
-  (segment (start 171.069 169.545) (end 172.085 169.545) (width 0.1524) (layer In2.Cu) (net 3))
-  (segment (start 172.085 169.545) (end 175.26 172.72) (width 0.1524) (layer In2.Cu) (net 3))
-  (segment (start 175.69998 184.94912) (end 175.69998 180.77998) (width 0.1524) (layer B.Cu) (net 3))
-  (segment (start 175.69998 180.77998) (end 175.26 180.34) (width 0.1524) (layer B.Cu) (net 3))
-  (segment (start 176.6982 184.94912) (end 176.6982 181.7782) (width 0.1524) (layer B.Cu) (net 3))
-  (segment (start 176.6982 181.7782) (end 175.26 180.34) (width 0.1524) (layer B.Cu) (net 3))
-  (via (at 175.26 180.34) (size 0.4572) (drill 0.254) (layers F.Cu B.Cu) (net 3))
-  (segment (start 175.26 180.34) (end 175.69998 180.77998) (width 0.1524) (layer F.Cu) (net 3))
-  (segment (start 174.69922 180.90078) (end 175.26 180.34) (width 0.1524) (layer F.Cu) (net 3))
-  (segment (start 174.69922 184.94912) (end 174.69922 180.90078) (width 0.1524) (layer F.Cu) (net 3))
-  (segment (start 175.69998 184.94912) (end 175.69998 180.77998) (width 0.1524) (layer F.Cu) (net 3))
-  (segment (start 175.69998 180.77998) (end 176.6982 181.7782) (width 0.1524) (layer F.Cu) (net 3))
-  (segment (start 176.6982 181.7782) (end 176.6982 184.94912) (width 0.1524) (layer F.Cu) (net 3))
+  (segment (start 175.26 178.520341) (end 174.675795 179.104543) (width 0.1524) (layer In2.Cu) (net 3))
+  (segment (start 175.26 172.72) (end 175.26 178.520341) (width 0.1524) (layer In2.Cu) (net 3))
+  (segment (start 174.675795 179.104543) (end 174.675795 180.051454) (width 0.1524) (layer In2.Cu) (net 3))
+  (segment (start 174.989742 180.57777) (end 175.793401 181.381429) (width 0.1524) (layer In2.Cu) (net 3))
+  (segment (start 166.624 169.418) (end 166.624 171.999659) (width 0.1524) (layer In2.Cu) (net 3))
+  (segment (start 166.624 171.999659) (end 174.989742 180.365401) (width 0.1524) (layer In2.Cu) (net 3))
+  (segment (start 174.989742 180.365401) (end 174.989742 180.57777) (width 0.1524) (layer In2.Cu) (net 3))
+  (segment (start 174.675795 180.051454) (end 174.989742 180.365401) (width 0.1524) (layer In2.Cu) (net 3))
+  (segment (start 175.793401 181.381429) (end 176.022 181.610028) (width 0.1524) (layer In2.Cu) (net 3))
+  (segment (start 175.69998 184.94912) (end 175.69998 181.93202) (width 0.1524) (layer F.Cu) (net 3))
+  (segment (start 175.69998 181.93202) (end 176.022 181.61) (width 0.1524) (layer F.Cu) (net 3))
+  (segment (start 176.022 181.61) (end 176.6982 182.2862) (width 0.1524) (layer F.Cu) (net 3))
+  (segment (start 176.6982 182.2862) (end 176.6982 184.94912) (width 0.1524) (layer F.Cu) (net 3))
+  (segment (start 176.022 181.61) (end 176.022 181.610028) (width 0.1524) (layer F.Cu) (net 3))
+  (segment (start 175.69998 184.94912) (end 175.69998 181.93202) (width 0.1524) (layer B.Cu) (net 3))
+  (segment (start 175.69998 181.93202) (end 176.022 181.61) (width 0.1524) (layer B.Cu) (net 3))
+  (segment (start 176.022 181.61) (end 176.6982 182.2862) (width 0.1524) (layer B.Cu) (net 3))
+  (segment (start 176.6982 182.2862) (end 176.6982 184.94912) (width 0.1524) (layer B.Cu) (net 3))
+  (segment (start 176.022 181.61) (end 176.022 181.610028) (width 0.1524) (layer B.Cu) (net 3))
+  (segment (start 174.69922 182.97427) (end 176.022 181.65149) (width 0.1524) (layer F.Cu) (net 3))
+  (segment (start 174.69922 184.94912) (end 174.69922 182.97427) (width 0.1524) (layer F.Cu) (net 3))
+  (segment (start 176.022 181.65149) (end 176.022 181.610028) (width 0.1524) (layer F.Cu) (net 3))
+  (via (at 176.022 181.610028) (size 0.4572) (drill 0.254) (layers F.Cu B.Cu) (net 3))
   (segment (start 174.69922 184.94912) (end 174.69922 181.080779) (width 0.1524) (layer F.Cu) (net 3))
   (segment (start 175.69998 187.25036) (end 175.69998 184.94912) (width 0.1524) (layer B.Cu) (net 3))
@@
   (segment (start 167.259 173.736) (end 167.259 176.276) (width 0.1524) (layer F.Cu) (net 3))
   (segment (start 167.259 176.276) (end 167.259 178.816) (width 0.1524) (layer F.Cu) (net 3))
-  (segment (start 166.624 169.418) (end 166.751 169.545) (width 0.1524) (layer In2.Cu) (net 3))
-  (segment (start 166.751 169.545) (end 171.069 169.545) (width 0.1524) (layer In2.Cu) (net 3))
   (segment (start 166.624 169.418) (end 166.624 169.799) (width 0.1524) (layer F.Cu) (net 3))
   (segment (start 166.624 169.799) (end 167.259 170.434) (width 0.1524) (layer F.Cu) (net 3))
   (segment (start 167.259 170.434) (end 167.259 173.736) (width 0.1524) (layer F.Cu) (net 3))
   (segment (start 171.069 169.545) (end 166.751 169.545) (width 0.1524) (layer In2.Cu) (net 3))
+  (segment (start 183.69844 184.94912) (end 183.69844 180.160051) (width 0.1524) (layer B.Cu) (net 4))
+  (segment (start 183.69844 180.160051) (end 183.600813 180.062424) (width 0.1524) (layer B.Cu) (net 4))
   (segment (start 190.754 163.322) (end 190.754 165.1) (width 0.4572) (layer In2.Cu) (net 4))
   (segment (start 189.484 162.052) (end 190.754 163.322) (width 0.4572) (layer In2.Cu) (net 4))
@@
   )
   (zone (net 59) (net_name /VCC5V0) (layer In2.Cu) (hatch edge 0.508)
-    (priority 2)
+    (priority 1)
     (connect_pads (clearance 0.254))
     (min_thickness 0.254)
@@
   )
   (zone (net 4) (net_name /VCC3V3) (layer In2.Cu) (hatch edge 0.508)
-    (priority 1)
+    (priority 2)
     (connect_pads (clearance 0.254))
     (min_thickness 0.254)

Commit message: Temp commit.
Routing:
- net /N_LVDS_1_N: track 21.7 -> 30.6 mm
- net /N_LVDS_1_P: track 25.1 -> 32.7 mm
- net /N_LVDS_2_N: track 25.4 -> 32.7 mm
- net /N_LVDS_2_P: track 24.6 -> 31.0 mm
- net /N_SCL: track 65.7 -> 62.1 mm
- net /S_LVDS_0_P: track 27.6 -> 30.5 mm
- net /N_SDA: track 69.5 -> 69.0 mm
